File: kicad/amplifier/amplifier.sch (KiCad schematic (older format))
At the start: 25 parts, among them J1 Audio In, J2 Speaker, J3 Jack-DC 15v, J4 +12v, J5 GND1, SW1 On/Off, U1 TDA2003, U2 L7812

Commit message: Power supply modifications
Parts:
- added C11: 220nF, symbol Device:C
- added C12: 100nF, symbol Device:C
- added J6: +5v, symbol Connector_Generic:Conn_01x03
- added J7: 5v/GND2, symbol Connector_Generic:Conn_01x02
- added U3: MP2307_Breakout, symbol CostumParts:MP2307_Breakout
- added U4: L7805, symbol Regulator_Linear:L7805
- added U5: PQS07-S5-S5, symbol CostumParts:PQS07-S5-S5
Connections:
- net labels added: +5V, +8v, GND2
- wire segments 68 -> 86
Other:
- moved on the sheet: C10, C9, J3, SW1, U2
